File: h7-disco.brd (EAGLE design)
At the start: 85.6 x 94 mm, 123 parts, among them CN2 M06X2, J1 CONN_25X2, J2 CONN_25X2, J3 ULPI, J4 BOOT0, J5 ST-LINK, J6 +3V3, J9 SWD, Q1 8 MHz, Q2 32KHz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

Commit message: Elements value fix.
Parts:
- C11: value 2.2uF -> 100nF
- C24, C5: value 0.33µF -> 100nF
- C25: value 2.2uF -> 0.1uF
- C26: value 2.2uF -> 1µF
- R1, R11, R3, R33: value (none) -> 100K
- R2, R21, R22, R34: value (none) -> 10K
- R30: value (none) -> 4K7
- R4, R5: value (none) -> 22
Changed lines of the file:
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@@
 <attribute name="VALUE" x="45.72" y="57.531" size="0.6096" layer="27" font="vector" ratio="20" rot="R270" align="top-center"/>
 </element>
-<element name="C5" library="SparkFun-Capacitors" package="0805" value="0.33µF" x="13.589" y="8.3185" smashed="yes" rot="R180">
+<element name="C5" library="SparkFun-Capacitors" package="0805" value="100nF" x="13.589" y="8.3185" smashed="yes" rot="R180">
 <attribute name="PROD_ID" value="CAP-08469" x="13.589" y="8.3185" size="1.778" layer="27" rot="R180" display="off"/>
 <attribute name="NAME" x="13.335" y="7.3025" size="0.8128" layer="25" font="vector" ratio="20" rot="R180" align="bottom-center"/>
@@
 <attribute name="VALUE" x="46.482" y="50.927" size="1.27" layer="27" ratio="10" rot="R90"/>
 </element>
-<element name="R1" library="SparkFun-Resistors" package="0805" value=" " x="15.748" y="52.705" smashed="yes" rot="R90">
+<element name="R1" library="SparkFun-Resistors" package="0805" value="100K" x="15.748" y="52.705" smashed="yes" rot="R90">
 <attribute name="PROD_ID" value=" " x="15.748" y="52.705" size="1.778" layer="27" rot="R90" display="off"/>
 <attribute name="NAME" x="14.7955" y="52.705" size="0.8128" layer="25" font="vector" ratio="20" rot="R90" align="bottom-center"/>
 <attribute name="VALUE" x="16.637" y="52.705" size="0.6096" layer="27" font="vector" ratio="20" rot="R90" align="top-center"/>
 </element>
-<element name="R2" library="SparkFun-Resistors" package="0805" value=" " x="49.149" y="38.354" smashed="yes" rot="R90">
+<element name="R2" library="SparkFun-Resistors" package="0805" value="10K" x="49.149" y="38.354" smashed="yes" rot="R90">
 <attribute name="PROD_ID" value=" " x="49.149" y="38.354" size="1.778" layer="27" rot="R90" display="off"/>
 <attribute name="NAME" x="48.133" y="37.9095" size="0.8128" layer="25" font="vector" ratio="20" rot="R90" align="bottom-center"/>
 <attribute name="VALUE" x="50.038" y="38.354" size="0.6096" layer="27" font="vector" ratio="20" rot="R90" align="top-center"/>
 </element>
-<element name="R3" library="SparkFun-Resistors" package="0805" value=" " x="23.114" y="6.35" smashed="yes" rot="R270">
+<element name="R3" library="SparkFun-Resistors" package="0805" value="100K" x="23.114" y="6.35" smashed="yes" rot="R270">
 <attribute name="PROD_ID" value=" " x="23.114" y="6.35" size="1.778" layer="27" rot="R270" display="off"/>
 <attribute name="NAME" x="24.13" y="6.2865" size="0.8128" layer="25" font="vector" ratio="20" rot="R270" align="bottom-center"/>
@@
 <attribute name="VALUE" x="35.814" y="83.82" size="0.6096" layer="27" font="vector" ratio="20" rot="R270" align="top-center"/>
 </element>
-<element name="C24" library="SparkFun-Capacitors" package="0805" value="0.33µF" x="8.255" y="90.17" smashed="yes" rot="R270">
+<element name="C24" library="SparkFun-Capacitors" package="0805" value="100nF" x="8.255" y="90.17" smashed="yes" rot="R270">
 <attribute name="PROD_ID" value="CAP-08469" x="8.255" y="90.17" size="1.778" layer="27" rot="R270" display="off"/>
 <attribute name="VALUE" value="0.33µF" x="8.255" y="90.17" size="1.778" layer="27" rot="R270" display="off"/>
@@
 <attribute name="VALUE" x="39.878" y="83.185" size="0.6096" layer="27" font="vector" ratio="20" rot="R90" align="top-center"/>
 </element>
-<element name="C25" library="SparkFun-Capacitors" package="0805" value="2.2uF" x="14.986" y="90.17" smashed="yes" rot="R90">
+<element name="C25" library="SparkFun-Capacitors" package="0805" value="0.1uF" x="14.986" y="90.17" smashed="yes" rot="R90">
 <attribute name="PROD_ID" value="CAP-11624" x="14.986" y="90.17" size="1.778" layer="27" rot="R90" display="off"/>
 <attribute name="VALUE" value="2.2uF" x="14.986" y="90.17" size="1.778" layer="27" rot="R90" display="off"/>
@@
 <attribute name="VALUE" x="15.875" y="90.17" size="0.6096" layer="27" font="vector" ratio="20" rot="R90" align="top-center"/>
 </element>
-<element name="C11" library="SparkFun-Capacitors" package="0805" value="2.2uF" x="38.354" y="90.932" smashed="yes" rot="R90">
+<element name="C11" library="SparkFun-Capacitors" package="0805" value="100nF" x="38.354" y="90.932" smashed="yes" rot="R90">
 <attribute name="PROD_ID" value="CAP-11624" x="38.354" y="90.932" size="1.778" layer="27" rot="R90" display="off"/>
 <attribute name="VALUE" value="2.2uF" x="38.354" y="90.932" size="1.778" layer="27" rot="R90" display="off"/>
@@
 <attribute name="VALUE" x="35.052" y="87.376" size="0.6096" layer="27" font="vector" ratio="20" rot="R270" align="top-center"/>
 </element>
-<element name="R11" library="SparkFun-Resistors" package="0805" value=" " x="38.354" y="87.376" smashed="yes" rot="R270">
+<element name="R11" library="SparkFun-Resistors" package="0805" value="100K" x="38.354" y="87.376" smashed="yes" rot="R270">
 <attribute name="PROD_ID" value=" " x="38.354" y="87.376" size="1.778" layer="27" rot="R270" display="off"/>
 <attribute name="VALUE" value=" " x="38.354" y="87.376" size="1.778" layer="27" rot="R270" display="off"/>
@@
 <attribute name="VALUE" x="17.907" y="88.138" size="0.6096" layer="27" font="vector" ratio="20" rot="R180" align="top-center"/>
 </element>
-<element name="R21" library="SparkFun-Resistors" package="0805" value=" " x="37.084" y="76.073" smashed="yes" rot="R90">
+<element name="R21" library="SparkFun-Resistors" package="0805" value="10K" x="37.084" y="76.073" smashed="yes" rot="R90">
 <attribute name="PROD_ID" value=" " x="37.084" y="76.073" size="1.778" layer="27" rot="R90" display="off"/>
 <attribute name="VALUE" value=" " x="37.084" y="76.073" size="1.778" layer="27" rot="R90" display="off"/>
@@
 <attribute name="VALUE" x="37.973" y="76.073" size="0.6096" layer="27" font="vector" ratio="20" rot="R90" align="top-center"/>
 </element>
-<element name="R22" library="SparkFun-Resistors" package="0805" value=" " x="39.37" y="76.073" smashed="yes" rot="R270">
+<element name="R22" library="SparkFun-Resistors" package="0805" value="10K" x="39.37" y="76.073" smashed="yes" rot="R270">
 <attribute name="PROD_ID" value=" " x="39.37" y="76.073" size="1.778" layer="27" rot="R270" display="off"/>
 <attribute name="VALUE" value=" " x="39.37" y="76.073" size="1.778" layer="27" rot="R270" display="off"/>
@@
 <attribute name="VALUE" x="17.272" y="80.264" size="0.6096" layer="27" font="vector" ratio="20" rot="R90" align="top-center"/>
 </element>
-<element name="R30" library="SparkFun-Resistors" package="0805" value=" " x="31.115" y="75.565" smashed="yes">
+<element name="R30" library="SparkFun-Resistors" package="0805" value="4K7" x="31.115" y="75.565" smashed="yes">
 <attribute name="PROD_ID" value=" " x="31.115" y="75.565" size="1.778" layer="27" display="off"/>
 <attribute name="VALUE" value=" " x="31.115" y="75.565" size="1.778" layer="27" display="off"/>
@@
 <attribute name="VALUE" x="31.115" y="74.676" size="0.6096" layer="27" font="vector" ratio="20" align="top-center"/>
 </element>
-<element name="R4" library="SparkFun-Resistors" package="0805" value=" " x="12.573" y="84.074" smashed="yes">
+<element name="R4" library="SparkFun-Resistors" package="0805" value="22" x="12.573" y="84.074" smashed="yes">
 <attribute name="PROD_ID" value=" " x="12.573" y="84.074" size="1.778" layer="27" display="off"/>
 <attribute name="VALUE" value=" " x="12.573" y="84.074" size="1.778" layer="27" display="off"/>
@@
 <attribute name="VALUE" x="12.573" y="83.185" size="0.6096" layer="27" font="vector" ratio="20" align="top-center"/>
 </element>
-<element name="R5" library="SparkFun-Resistors" package="0805" value=" " x="12.573" y="81.661" smashed="yes">
+<element name="R5" library="SparkFun-Resistors" package="0805" value="22" x="12.573" y="81.661" smashed="yes">
 <attribute name="PROD_ID" value=" " x="12.573" y="81.661" size="1.778" layer="27" display="off"/>
 <attribute name="VALUE" value=" " x="12.573" y="81.661" size="1.778" layer="27" display="off"/>
@@
 <attribute name="VALUE" x="8.98525" y="78.20025" size="0.6096" layer="27" font="vector" ratio="20" rot="R270" align="top-center"/>
 </element>
-<element name="C26" library="SparkFun-Capacitors" package="1206" value="2.2uF" x="3.84175" y="89.4715" smashed="yes">
+<element name="C26" library="SparkFun-Capacitors" package="1206" value="1µF" x="3.84175" y="89.4715" smashed="yes">
 <attribute name="PROD_ID" value="CAP-10009" x="3.84175" y="89.4715" size="1.778" layer="27" display="off"/>
 <attribute name="VALUE" value="2.2uF" x="3.84175" y="89.4715" size="1.778" layer="27" display="off"/>
@@
 <attribute name="VALUE" x="69.469" y="33.401" size="0.6096" layer="28" font="vector" ratio="20" rot="MR90" align="top-center"/>
 </element>
-<element name="R33" library="SparkFun-Resistors" package="0805" value=" " x="70.6755" y="41.8465" smashed="yes" rot="MR90">
+<element name="R33" library="SparkFun-Resistors" package="0805" value="100K" x="70.6755" y="41.8465" smashed="yes" rot="MR90">
 <attribute name="PROD_ID" value=" " x="70.6755" y="41.8465" size="1.778" layer="28" rot="MR90" display="off"/>
 <attribute name="NAME" x="71.6915" y="42.8625" size="0.8128" layer="26" font="vector" ratio="15" rot="MR90" align="bottom-center"/>
@@
 <attribute name="VALUE" x="71.5645" y="45.6565" size="0.6096" layer="28" font="vector" ratio="20" rot="MR270" align="top-center"/>
 </element>
-<element name="R34" library="SparkFun-Resistors" package="0805" value=" " x="76.581" y="44.3865" smashed="yes" rot="MR0">
+<element name="R34" library="SparkFun-Resistors" package="0805" value="10K" x="76.581" y="44.3865" smashed="yes" rot="MR0">
 <attribute name="PROD_ID" value=" " x="76.581" y="44.3865" size="1.778" layer="28" rot="MR0" display="off"/>
 <attribute name="NAME" x="74.8665" y="44.3865" size="0.8128" layer="26" font="vector" ratio="20" rot="MR270" align="bottom-center"/>

Commit message: add MCO pin
Parts:
- added MCO: TPTP10R, testpad:TP10R
- C13, C14: value 0.1µF -> 2.2µF
- C23: value 10nF -> 1µF; device SparkFun-Capacitors:0805 -> SparkFun-Capacitors:1206
- moved C23 38.1 mm to (22.7, 55.2), turned to 180 degrees
- moved R9 3.17 mm to (27.0, 89.5), turned to 90 degrees
- moved R8 2.29 mm to (35.9, 90.9)
- moved C19 1.99 mm to (29.5, 89.5), turned to 90 degrees
- moved T_JTDI 1.68 mm to (32.1, 89.2)
- moved AIN_1 1.37 mm to (33.6, 89.2)
- moved PWR_ENN 0.80 mm to (24.4, 89.9)
Connections:
- new net MCO: MCO.TP, STM32F103CB.29
- net +5V: now also C23.2
- net AIN_1: no longer C23.1
- net GND: now also C23.1
- net ST_GND: no longer C23.2
Routing:
- net N$25: track 0.00 -> 66.2 mm
- net MCO: track 0.00 -> 6.63 mm
- net GND: track 755.8 -> 760.3 mm, vias 21 -> 22
- net +5V: track 106.3 -> 110.0 mm
- net AIN_1: track 12.4 -> 9.20 mm
- net T_JTMS: track 30.3 -> 33.1 mm
- net T_NRST: track 24.5 -> 22.1 mm
- net T_SWDIO_IN: track 2.16 -> 4.29 mm
- net ST_GND: track 212.6 -> 214.7 mm
- net ST_+3V3: track 91.2 -> 90.5 mm

Commit message: improve
Parts:
- R35: value (none) -> 100K
- moved R40 3.05 mm to (74.7, 14.2)
Routing:
- net N$21: track 7.97 -> 9.87 mm
- net PC13_: track 19.3 -> 18.7 mm
Changed lines of the file:
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@@
 <attribute name="VALUE" x="73.0885" y="9.652" size="0.4064" layer="28" rot="MR0"/>
 </element>
-<element name="R35" library="SparkFun-Resistors" package="0805" value=" " x="74.4855" y="4.445" smashed="yes" rot="MR180">
+<element name="R35" library="SparkFun-Resistors" package="0805" value="100K" x="74.4855" y="4.445" smashed="yes" rot="MR180">
 <attribute name="PROD_ID" value=" " x="74.4855" y="4.445" size="1.778" layer="28" rot="MR180" display="off"/>
 <attribute name="NAME" x="72.9615" y="3.3655" size="0.8128" layer="26" font="vector" ratio="15" rot="MR180" align="bottom-center"/>
@@
 <attribute name="VALUE" x="76.708" y="16.8275" size="0.6096" layer="28" font="vector" ratio="20" rot="MR270" align="top-center"/>
 </element>
-<element name="R40" library="SparkFun-Resistors" package="0805" value="36K" x="71.628" y="14.351" smashed="yes">
-<attribute name="PROD_ID" value=" " x="51.308" y="25.781" size="1.778" layer="27" display="off"/>
-<attribute name="NAME" x="71.4375" y="15.3035" size="0.8128" layer="25" font="vector" ratio="15" align="bottom-center"/>
-<attribute name="VALUE" x="71.628" y="13.462" size="0.6096" layer="27" font="vector" ratio="20" align="top-center"/>
+<element name="R40" library="SparkFun-Resistors" package="0805" value="36K" x="74.676" y="14.224" smashed="yes">
+<attribute name="PROD_ID" value=" " x="54.356" y="25.654" size="1.778" layer="27" display="off"/>
+<attribute name="NAME" x="74.676" y="15.1765" size="0.8128" layer="25" font="vector" ratio="15" align="bottom-center"/>
+<attribute name="VALUE" x="74.676" y="13.335" size="0.6096" layer="27" font="vector" ratio="20" align="top-center"/>
 </element>
 <element name="R41" library="SparkFun-Resistors" package="0805" value="100" x="77.851" y="20.0025" smashed="yes" rot="MR90">
@@
 <wire x1="78.105" y1="6.9215" x2="77.0255" y2="8.001" width="0.4064" layer="1"/>
 <wire x1="77.0255" y1="8.001" x2="77.0255" y2="13.081" width="0.4064" layer="1"/>
-<wire x1="77.0255" y1="13.081" x2="70.739" y2="13.081" width="0.4064" layer="1"/>
-<wire x1="70.6755" y1="17.0815" x2="72.3265" y2="18.7325" width="0.254" layer="1"/>
-<wire x1="72.3265" y1="18.7325" x2="73.071284375" y2="19.470303125" width="0.254" layer="1"/>
+<wire x1="77.0255" y1="13.081" x2="73.66" y2="13.081" width="0.4064" layer="1"/>
+<wire x1="73.66" y1="13.081" x2="71.501" y2="13.081" width="0.4064" layer="1"/>
 <wire x1="66.8655" y1="2.4765" x2="67.3735" y2="1.9685" width="0.8128" layer="1"/>
 <wire x1="67.3735" y1="1.9685" x2="70.866" y2="1.9685" width="0.8128" layer="1"/>
@@
 <wire x1="69.0355" y1="48.1965" x2="66.8655" y2="48.1965" width="0.6096" layer="16"/>
 <contactref element="R40" pad="1"/>
-<wire x1="70.739" y1="13.081" x2="70.728" y2="13.07" width="0.254" layer="1"/>
-<wire x1="70.728" y1="14.351" x2="70.6755" y2="14.848" width="0.254" layer="1"/>
-<wire x1="70.6755" y1="14.848" x2="70.6755" y2="17.0815" width="0.254" layer="1"/>
-<wire x1="70.728" y1="13.07" x2="70.728" y2="14.351" width="0.4064" layer="1"/>
 <wire x1="76.8985" y1="4.699" x2="76.8985" y2="5.7785" width="0.6096" layer="16"/>
 <wire x1="76.8985" y1="5.7785" x2="76.962" y2="5.842" width="0.4064" layer="16"/>
@@
 <wire x1="26.162" y1="56.5785" x2="26.162" y2="58.3565" width="0.8128" layer="16"/>
 <wire x1="26.162" y1="58.3565" x2="26.2255" y2="58.42" width="0.8128" layer="16"/>
+<wire x1="71.501" y1="17.907" x2="71.501" y2="17.78" width="0.254" layer="1"/>
+<wire x1="73.071284375" y1="19.470303125" x2="72.33348125" y2="18.7325" width="0.254" layer="1"/>
+<wire x1="72.33348125" y1="18.7325" x2="71.501" y2="17.907" width="0.254" layer="1"/>
+<wire x1="71.501" y1="13.081" x2="71.501" y2="17.78" width="0.4064" layer="1"/>
+<wire x1="73.776" y1="14.224" x2="73.776" y2="13.197" width="0.4064" layer="1"/>
+<wire x1="73.776" y1="13.197" x2="73.66" y2="13.081" width="0.4064" layer="1"/>
 <wire x1="76.8985" y1="4.6355" x2="76.708" y2="4.445" width="0" layer="19" extent="1-16"/>
 <wire x1="76.8985" y1="4.699" x2="76.8985" y2="4.6355" width="0" layer="19" extent="1-1"/>
@@
 <wire x1="74.4855" y1="36.5125" x2="71.3105" y2="39.6875" width="0.3048" layer="1"/>
 <via x="71.3105" y="39.6875" extent="1-16" drill="0.3048"/>
-<wire x1="70.6755" y1="40.9465" x2="70.6755" y2="40.3225" width="0.6096" layer="16"/>
-<wire x1="70.6755" y1="40.3225" x2="71.3105" y2="39.6875" width="0.6096" layer="16"/>
 <wire x1="73.025" y1="47.8155" x2="71.1835" y2="47.8155" width="0.6096" layer="16"/>
 <wire x1="71.1835" y1="47.8155" x2="70.6755" y2="48.3235" width="0.6096" layer="16"/>
@@
 <wire x1="72.9615" y1="51.7525" x2="70.6755" y2="49.4665" width="0.6096" layer="16"/>
 <contactref element="T2" pad="3"/>
-<wire x1="71.3105" y1="39.6875" x2="72.1995" y2="40.5765" width="0.6096" layer="16"/>
-<wire x1="72.1995" y1="40.5765" x2="73.406" y2="40.5765" width="0.6096" layer="16"/>
 <wire x1="73.025" y1="47.8155" x2="73.406" y2="47.4345" width="0.6096" layer="16"/>
 <wire x1="73.406" y1="47.4345" x2="73.406" y2="40.5765" width="0.6096" layer="16"/>
@@
 <wire x1="71.671" y1="15.9815" x2="74.4855" y2="18.796" width="0.4064" layer="16"/>
 <wire x1="74.4855" y1="18.796" x2="74.4855" y2="18.923" width="0.254" layer="16"/>
+<wire x1="73.406" y1="40.5765" x2="71.501" y2="40.5765" width="0.6096" layer="16"/>
+<wire x1="71.501" y1="40.5765" x2="71.0455" y2="40.5765" width="0.6096" layer="16"/>
+<wire x1="71.0455" y1="40.5765" x2="70.6755" y2="40.9465" width="0.6096" layer="16"/>
+<wire x1="71.3105" y1="39.6875" x2="71.3105" y2="40.386" width="0.6096" layer="16"/>
+<wire x1="71.3105" y1="40.386" x2="71.501" y2="40.5765" width="0.6096" layer="16"/>
 <wire x1="60.452" y1="56.388" x2="66.8655" y2="50.7365" width="0" layer="19" extent="16-16"/>
 </signal>
@@
 <wire x1="72.5805" y1="29.153478125" x2="72.5805" y2="30.0355" width="0.254" layer="1"/>
 <wire x1="72.5805" y1="30.0355" x2="73.9775" y2="31.4325" width="0.254" layer="1"/>
-<wire x1="73.9775" y1="31.4325" x2="73.9775" y2="36.195" width="0.254" layer="1"/>
-<wire x1="73.9775" y1="36.195" x2="73.3425" y2="36.83" width="0.254" layer="1"/>
-<wire x1="73.3425" y1="36.83" x2="71.501" y2="36.83" width="0.254" layer="1"/>
-<wire x1="71.501" y1="36.83" x2="68.453" y2="39.878" width="0.254" layer="1"/>
-<wire x1="68.453" y1="39.878" x2="68.453" y2="41.529" width="0.254" layer="1"/>
-<wire x1="68.453" y1="41.529" x2="66.8655" y2="43.1165" width="0.254" layer="1"/>
+<wire x1="73.9775" y1="31.4325" x2="73.9775" y2="35.7505" width="0.254" layer="1"/>
+<wire x1="73.9775" y1="35.7505" x2="72.898" y2="36.83" width="0.254" layer="1"/>
+<wire x1="72.898" y1="36.83" x2="72.0725" y2="36.83" width="0.254" layer="1"/>
+<wire x1="72.0725" y1="36.83" x2="68.7705" y2="40.132" width="0.254" layer="1"/>
+<wire x1="68.7705" y1="40.132" x2="68.7705" y2="41.2115" width="0.254" layer="1"/>
+<wire x1="68.7705" y1="41.2115" x2="66.8655" y2="43.1165" width="0.254" layer="1"/>
 </signal>
 <signal name="N$24">
@@
 <wire x1="73.871" y1="16.825" x2="73.848" y2="16.825" width="0.254" layer="16"/>
 <wire x1="73.848" y1="16.825" x2="72.898" y2="15.875" width="0.254" layer="16"/>
-<wire x1="72.898" y1="15.875" x2="72.7075" y2="15.6845" width="0.254" layer="1"/>
-<wire x1="72.7075" y1="15.6845" x2="72.7075" y2="14.732" width="0.254" layer="1"/>
-<wire x1="72.7075" y1="14.732" x2="72.528" y2="14.5525" width="0.254" layer="1"/>
-<wire x1="72.528" y1="14.5525" x2="72.528" y2="14.351" width="0.254" layer="1"/>
+<wire x1="72.898" y1="15.875" x2="74.295" y2="15.875" width="0.254" layer="1"/>
 <wire x1="73.871" y1="16.825" x2="74.7735" y2="17.7275" width="0.254" layer="16"/>
 <wire x1="74.7735" y1="17.7275" x2="75.819" y2="17.7275" width="0.254" layer="16"/>
 <wire x1="75.819" y1="17.7275" x2="77.194" y2="19.1025" width="0.254" layer="16"/>
 <wire x1="77.194" y1="19.1025" x2="77.851" y2="19.1025" width="0.254" layer="16"/>
+<wire x1="74.295" y1="15.875" x2="75.576" y2="14.594" width="0.254" layer="1"/>
+<wire x1="75.576" y1="14.594" x2="75.576" y2="14.224" width="0.254" layer="1"/>
 </signal>
 <signal name="MCO">
