File: h7-disco.sch (EAGLE design)
At the start: 123 parts, among them CN2 M06X2, J1 CONN_25X2, J2 CONN_25X2, J3 ULPI, J4 BOOT0, J5 ST-LINK, J6 +3V3, J9 SWD, Q1 8 MHz, Q2 32KHz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

Commit message: Elements value fix.
Parts:
- C11: value 2.2uF -> 100nF
- C24, C5: value 0.33µF -> 100nF
- C25: value 2.2uF -> 0.1uF
- C26: value 2.2uF -> 1µF
- R1, R11, R3, R33: value (none) -> 100K
- R2, R21, R22, R34: value (none) -> 10K
- R30: value (none) -> 4K7
- R4, R5: value (none) -> 22
Other:
- moved on the sheet: R2

Commit message: add MCO pin
Parts:
- added MCO: TPTP10R, testpad:TPTP10R
- C13, C14: value 0.1µF -> 2.2µF
- C23: value 10nF -> 1µF; device SparkFun-Capacitors:2.2UF-0805-25V-(+80/-20%) -> SparkFun-Capacitors:2.2UF-1206-50V-10%
Connections:
- new net MCO: MCO.TP, STM32F103CBPORTA_H.PA8
- net +5V: now also C23.2
- net AIN_1: no longer C23.1
- net GND: now also C23.1
- net ST_GND: no longer C23.2
Other:
- moved on the sheet: C23, J3, U3

Commit message: improve
Parts:
- R35: value (none) -> 100K
Other:
- moved on the sheet: LED8
Changed lines of the file:
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@@
 <part name="USB_" library="con-hirose" deviceset="MICRO-USB-SHIELD-" device="MICRO_USB-B_4.85_HORN" value="usb"/>
 <part name="U3" library="SparkFun-IC-Power" deviceset="V_REG_LM1117" device="SOT223" value="LM1117-33"/>
-<part name="R35" library="SparkFun-Resistors" deviceset="RESISTOR" device="0805" value=" "/>
+<part name="R35" library="SparkFun-Resistors" deviceset="RESISTOR" device="0805" value="100K"/>
 <part name="GND36" library="supply1" deviceset="GND" device=""/>
 <part name="+3V20" library="supply1" deviceset="+3V3" device=""/>
@@
 <instance part="R11" gate="G$1" x="80.01" y="157.48"/>
 <instance part="+3V7" gate="G$1" x="90.17" y="157.48" smashed="yes" rot="R270">
-<attribute name="VALUE" x="90.424" y="160.782" size="1.778" layer="96" rot="R270"/>
+<attribute name="VALUE" x="87.376" y="154.178" size="1.778" layer="96"/>
 </instance>
 <instance part="C11" gate="G$1" x="74.93" y="143.51"/>
@@
 <instance part="STM32" gate="MCU" x="287.02" y="50.8"/>
 <instance part="STM32" gate="PWR" x="287.02" y="-10.16" rot="R90"/>
-<instance part="Q3" gate="G$1" x="256.54" y="33.02" rot="R90"/>
+<instance part="Q3" gate="G$1" x="256.54" y="33.02" smashed="yes" rot="R90">
+<attribute name="NAME" x="255.524" y="37.084" size="1.778" layer="95" rot="R90"/>
+<attribute name="VALUE" x="259.08" y="37.084" size="1.778" layer="96" rot="R90"/>
+</instance>
 <instance part="C27" gate="G$1" x="246.38" y="35.56" smashed="yes" rot="R90">
 <attribute name="NAME" x="246.888" y="37.211" size="1.778" layer="95" font="vector"/>
@@
 <attribute name="VALUE" x="259.08" y="25.4" size="1.778" layer="96"/>
 </instance>
-<instance part="Q5" gate="G$1" x="238.76" y="55.88" rot="R90"/>
+<instance part="Q5" gate="G$1" x="238.76" y="55.88" smashed="yes" rot="R90">
+<attribute name="NAME" x="237.744" y="59.69" size="1.778" layer="95" rot="R90"/>
+<attribute name="VALUE" x="241.3" y="59.69" size="1.778" layer="96" rot="R90"/>
+</instance>
 <instance part="C35" gate="G$1" x="231.14" y="53.34" smashed="yes" rot="R90">
 <attribute name="NAME" x="231.521" y="51.816" size="1.778" layer="95" font="vector" rot="R270"/>
@@
 </instance>
 <instance part="GND37" gate="1" x="223.52" y="45.72"/>
-<instance part="LED8" gate="G$1" x="320.04" y="-30.48" smashed="yes">
-<attribute name="NAME" x="322.834" y="-31.877" size="1.778" layer="95" font="vector"/>
-<attribute name="VALUE" x="322.834" y="-33.655" size="1.778" layer="96" font="vector" align="top-left"/>
+<instance part="LED8" gate="G$1" x="320.04" y="-27.94" smashed="yes">
+<attribute name="NAME" x="322.834" y="-29.337" size="1.778" layer="95" font="vector"/>
+<attribute name="VALUE" x="322.834" y="-31.115" size="1.778" layer="96" font="vector" align="top-left"/>
 </instance>
 <instance part="R36" gate="G$1" x="320.04" y="-17.78" rot="R270"/>
@@
 <pinref part="LED8" gate="G$1" pin="C"/>
 <pinref part="GND38" gate="1" pin="GND"/>
+<wire x1="320.04" y1="-33.02" x2="320.04" y2="-35.56" width="0.1524" layer="91"/>
 </segment>
 <segment>
@@
 <segment>
 <pinref part="J4" gate="G$1" pin="1"/>
-<wire x1="248.92" y1="2.54" x2="248.92" y2="-2.54" width="0.1524" layer="91"/>
-<wire x1="248.92" y1="-2.54" x2="246.38" y2="-2.54" width="0.1524" layer="91"/>
+<wire x1="248.92" y1="2.54" x2="248.92" y2="-3.556" width="0.1524" layer="91"/>
+<wire x1="248.92" y1="-3.556" x2="246.38" y2="-3.556" width="0.1524" layer="91"/>
 <pinref part="+3V19" gate="G$1" pin="+3V3"/>
-<wire x1="246.38" y1="-2.54" x2="246.38" y2="-7.62" width="0.1524" layer="91"/>
+<wire x1="246.38" y1="-3.556" x2="246.38" y2="-7.62" width="0.1524" layer="91"/>
 </segment>
 <segment>
@@
 <wire x1="248.92" y1="-73.66" x2="248.92" y2="-58.674" width="0.1524" layer="91"/>
 <pinref part="R38" gate="G$1" pin="2"/>
-<wire x1="248.92" y1="-58.674" x2="248.92" y2="-60.96" width="0.1524" layer="91"/>
-<junction x="248.92" y="-58.674"/>
 </segment>
 </net>
@@
 <pinref part="R36" gate="G$1" pin="2"/>
 <pinref part="LED8" gate="G$1" pin="A"/>
-<wire x1="320.04" y1="-22.86" x2="320.04" y2="-27.94" width="0.1524" layer="91"/>
+<wire x1="320.04" y1="-22.86" x2="320.04" y2="-25.4" width="0.1524" layer="91"/>
 </segment>
 </net>
